Commit message: Updated colors of the gazebo model

File: src/robotic_arm_description/urdf/robotic_arm.xacro (robot description, xacro)
@@ -4,4 +4,5 @@
 <xacro:include filename="$(find robotic_arm_description)/urdf/robotic_arm.trans" />
 <xacro:include filename="$(find robotic_arm_description)/urdf/robotic_arm_gazebo.xacro"/>
+<xacro:include filename="$(find robotic_arm_description)/urdf/robotic_arm.gazebo.xacro"/>
 <xacro:include filename="$(find robotic_arm_description)/urdf/robotic_arm_controllers.xacro"/>
 <!-- Properties -->
@@ -9,7 +10,7 @@
 <link name="base_link">
   <inertial>
-    <origin xyz="0.2975 -0.19749999999999993 0.0075000000000000015" rpy="0 0 0"/>
-    <mass value="2.5415632831137143"/>
-    <inertia ixx="0.033087" iyy="0.075016" izz="0.108008" ixy="0.0" iyz="0.0" ixz="-0.0"/>
+    <origin xyz="4.1292719567255465e-17 -0.1275 0.0075" rpy="0 0 0"/>
+    <mass value="2.5408670074548567"/>
+    <inertia ixx="0.033061" iyy="0.074955" izz="0.107921" ixy="-0.0" iyz="0.0" ixz="0.0"/>
   </inertial>
   <visual>
@@ -29,10 +30,10 @@
 <link name="base_v2_1">
   <inertial>
-    <origin xyz="3.307089559423382e-07 -0.06999939486232204 0.0513656205942673" rpy="0 0 0"/>
+    <origin xyz="3.307089559204383e-07 -0.06999939486232201 0.0513656205942673" rpy="0 0 0"/>
     <mass value="0.5102582987586253"/>
     <inertia ixx="0.001541" iyy="0.00162" izz="0.002267" ixy="0.0" iyz="0.0" ixz="0.0"/>
   </inertial>
   <visual>
-    <origin xyz="-0.2975 0.0 -0.015" rpy="0 0 0"/>
+    <origin xyz="-0.0 -0.07 -0.015" rpy="0 0 0"/>
     <geometry>
       <mesh filename="package://robotic_arm_description/meshes/base_v2_1.stl" scale="0.001 0.001 0.001"/>
@@ -41,5 +42,5 @@
   </visual>
   <collision>
-    <origin xyz="-0.2975 0.0 -0.015" rpy="0 0 0"/>
+    <origin xyz="-0.0 -0.07 -0.015" rpy="0 0 0"/>
     <geometry>
       <mesh filename="package://robotic_arm_description/meshes/base_v2_1.stl" scale="0.001 0.001 0.001"/>
@@ -49,10 +50,10 @@
 <link name="waist_v6_1">
   <inertial>
-    <origin xyz="-0.00731793422720689 -0.0014787118544256073 0.019240916153628926" rpy="0 0 0"/>
+    <origin xyz="-0.007317934227206862 -0.0014787118544255873 0.019240916153628926" rpy="0 0 0"/>
     <mass value="0.08011233502112002"/>
     <inertia ixx="7.4e-05" iyy="5.5e-05" izz="6.5e-05" ixy="-0.0" iyz="7e-06" ixz="7e-06"/>
   </inertial>
   <visual>
-    <origin xyz="-0.2975 0.07 -0.101" rpy="0 0 0"/>
+    <origin xyz="-0.0 -0.0 -0.101" rpy="0 0 0"/>
     <geometry>
       <mesh filename="package://robotic_arm_description/meshes/waist_v6_1.stl" scale="0.001 0.001 0.001"/>
@@ -61,5 +62,5 @@
   </visual>
   <collision>
-    <origin xyz="-0.2975 0.07 -0.101" rpy="0 0 0"/>
+    <origin xyz="-0.0 -0.0 -0.101" rpy="0 0 0"/>
     <geometry>
       <mesh filename="package://robotic_arm_description/meshes/waist_v6_1.stl" scale="0.001 0.001 0.001"/>
@@ -69,10 +70,10 @@
 <link name="servomotormg996r_v2_2">
   <inertial>
-    <origin xyz="-0.01005433656255239 0.020152986183403193 -0.013081986774102439" rpy="0 0 0"/>
+    <origin xyz="-0.010054336562552477 0.020152986183403273 -0.013081986774102439" rpy="0 0 0"/>
     <mass value="0.2658706317147462"/>
     <inertia ixx="4.7e-05" iyy="6.1e-05" izz="6.1e-05" ixy="2e-06" iyz="1.5e-05" ixz="-2e-06"/>
   </inertial>
   <visual>
-    <origin xyz="-0.2795 0.097168 -0.147467" rpy="0 0 0"/>
+    <origin xyz="0.018 0.027168 -0.147467" rpy="0 0 0"/>
     <geometry>
       <mesh filename="package://robotic_arm_description/meshes/servomotormg996r_v2_2.stl" scale="0.001 0.001 0.001"/>
@@ -81,5 +82,5 @@
   </visual>
   <collision>
-    <origin xyz="-0.2795 0.097168 -0.147467" rpy="0 0 0"/>
+    <origin xyz="0.018 0.027168 -0.147467" rpy="0 0 0"/>
     <geometry>
       <mesh filename="package://robotic_arm_description/meshes/servomotormg996r_v2_2.stl" scale="0.001 0.001 0.001"/>
@@ -89,10 +90,10 @@
 <link name="link_1_v5_1">
   <inertial>
-    <origin xyz="0.007817729878361601 -2.3605874380216996e-07 0.05999982401434481" rpy="0 0 0"/>
+    <origin xyz="0.0078177298783616 -2.360587438056394e-07 0.05999982401434481" rpy="0 0 0"/>
     <mass value="0.07112302510728019"/>
     <inertia ixx="0.000121" iyy="0.000116" izz="1e-05" ixy="0.0" iyz="-0.0" ixz="0.0"/>
   </inertial>
   <visual>
-    <origin xyz="-0.2935 0.08391 -0.14128" rpy="0 0 0"/>
+    <origin xyz="0.004 0.01391 -0.14128" rpy="0 0 0"/>
     <geometry>
       <mesh filename="package://robotic_arm_description/meshes/link_1_v5_1.stl" scale="0.001 0.001 0.001"/>
@@ -101,5 +102,5 @@
   </visual>
   <collision>
-    <origin xyz="-0.2935 0.08391 -0.14128" rpy="0 0 0"/>
+    <origin xyz="0.004 0.01391 -0.14128" rpy="0 0 0"/>
     <geometry>
       <mesh filename="package://robotic_arm_description/meshes/link_1_v5_1.stl" scale="0.001 0.001 0.001"/>
@@ -109,10 +110,10 @@
 <link name="link_2a_v4_1">
   <inertial>
-    <origin xyz="-0.0057012559046490385 -0.04181110897598471 -3.1124321273889866e-05" rpy="0 0 0"/>
+    <origin xyz="-0.005701255904649023 -0.04181110897598475 -3.112432127394538e-05" rpy="0 0 0"/>
     <mass value="0.05167009815655824"/>
     <inertia ixx="6e-05" iyy="1e-05" izz="5.6e-05" ixy="0.0" iyz="-0.0" ixz="0.0"/>
   </inertial>
   <visual>
-    <origin xyz="-0.2935 0.08391 -0.26128" rpy="0 0 0"/>
+    <origin xyz="0.004 0.01391 -0.26128" rpy="0 0 0"/>
     <geometry>
       <mesh filename="package://robotic_arm_description/meshes/link_2a_v4_1.stl" scale="0.001 0.001 0.001"/>
@@ -121,5 +122,5 @@
   </visual>
   <collision>
-    <origin xyz="-0.2935 0.08391 -0.26128" rpy="0 0 0"/>
+    <origin xyz="0.004 0.01391 -0.26128" rpy="0 0 0"/>
     <geometry>
       <mesh filename="package://robotic_arm_description/meshes/link_2a_v4_1.stl" scale="0.001 0.001 0.001"/>
@@ -129,10 +130,10 @@
 <link name="link_2b_v4_1">
   <inertial>
-    <origin xyz="-0.008613311986319927 -0.017710429447622716 -4.645155661608946e-05" rpy="0 0 0"/>
+    <origin xyz="-0.008613311986319927 -0.017710429447622786 -4.6451556616200484e-05" rpy="0 0 0"/>
     <mass value="0.017891783436233155"/>
     <inertia ixx="5e-06" iyy="3e-06" izz="4e-06" ixy="1e-06" iyz="0.0" ixz="-0.0"/>
   </inertial>
   <visual>
-    <origin xyz="-0.3015 0.17366 -0.26128" rpy="0 0 0"/>
+    <origin xyz="-0.004 0.10366 -0.26128" rpy="0 0 0"/>
     <geometry>
       <mesh filename="package://robotic_arm_description/meshes/link_2b_v4_1.stl" scale="0.001 0.001 0.001"/>
@@ -141,5 +142,5 @@
   </visual>
   <collision>
-    <origin xyz="-0.3015 0.17366 -0.26128" rpy="0 0 0"/>
+    <origin xyz="-0.004 0.10366 -0.26128" rpy="0 0 0"/>
     <geometry>
       <mesh filename="package://robotic_arm_description/meshes/link_2b_v4_1.stl" scale="0.001 0.001 0.001"/>
@@ -149,10 +150,10 @@
 <link name="servomotormg996r_v2_3">
   <inertial>
-    <origin xyz="-0.010054336562552446 0.024498917400786344 0.005000000417687334" rpy="0 0 0"/>
+    <origin xyz="-0.010054336562552536 0.024498917400786264 0.005000000417687334" rpy="0 0 0"/>
     <mass value="0.2658706317147462"/>
     <inertia ixx="4.7e-05" iyy="4.6e-05" izz="7.5e-05" ixy="-2e-06" iyz="-0.0" ixz="-0.0"/>
   </inertial>
   <visual>
-    <origin xyz="-0.2825 0.11866 -0.25628" rpy="0 0 0"/>
+    <origin xyz="0.015 0.04866 -0.25628" rpy="0 0 0"/>
     <geometry>
       <mesh filename="package://robotic_arm_description/meshes/servomotormg996r_v2_3.stl" scale="0.001 0.001 0.001"/>
@@ -161,5 +162,5 @@
   </visual>
   <collision>
-    <origin xyz="-0.2825 0.11866 -0.25628" rpy="0 0 0"/>
+    <origin xyz="0.015 0.04866 -0.25628" rpy="0 0 0"/>
     <geometry>
       <mesh filename="package://robotic_arm_description/meshes/servomotormg996r_v2_3.stl" scale="0.001 0.001 0.001"/>
@@ -169,10 +170,10 @@
 <link name="servomotormicro9g_v2_1">
   <inertial>
-    <origin xyz="-0.005541210223247384 0.013371159759380885 -1.1102230246251565e-16" rpy="0 0 0"/>
+    <origin xyz="-0.005541210223247456 0.013371159759380774 -2.7755575615628914e-16" rpy="0 0 0"/>
     <mass value="0.05595068017526718"/>
     <inertia ixx="3e-06" iyy="4e-06" izz="6e-06" ixy="0.0" iyz="0.0" ixz="0.0"/>
   </inertial>
   <visual>
-    <origin xyz="-0.291 0.21046 -0.26128" rpy="0 0 0"/>
+    <origin xyz="0.0065 0.14046 -0.26128" rpy="0 0 0"/>
     <geometry>
       <mesh filename="package://robotic_arm_description/meshes/servomotormicro9g_v2_1.stl" scale="0.001 0.001 0.001"/>
@@ -181,5 +182,5 @@
   </visual>
   <collision>
-    <origin xyz="-0.291 0.21046 -0.26128" rpy="0 0 0"/>
+    <origin xyz="0.0065 0.14046 -0.26128" rpy="0 0 0"/>
     <geometry>
       <mesh filename="package://robotic_arm_description/meshes/servomotormicro9g_v2_1.stl" scale="0.001 0.001 0.001"/>
@@ -189,10 +190,10 @@
 <link name="gripper_base_v8_1">
   <inertial>
-    <origin xyz="0.011837914619012735 -0.02831046923426528 0.0067063756079010495" rpy="0 0 0"/>
+    <origin xyz="0.011837914619012749 -0.02831046923426539 0.006706375607900994" rpy="0 0 0"/>
     <mass value="0.020668522851976897"/>
     <inertia ixx="9e-06" iyy="4e-06" izz="1.1e-05" ixy="2e-06" iyz="1e-06" ixz="-0.0"/>
   </inertial>
   <visual>
-    <origin xyz="-0.3015 0.20166 -0.26128" rpy="0 0 0"/>
+    <origin xyz="-0.004 0.13166 -0.26128" rpy="0 0 0"/>
     <geometry>
       <mesh filename="package://robotic_arm_description/meshes/gripper_base_v8_1.stl" scale="0.001 0.001 0.001"/>
@@ -201,5 +202,5 @@
   </visual>
   <collision>
-    <origin xyz="-0.3015 0.20166 -0.26128" rpy="0 0 0"/>
+    <origin xyz="-0.004 0.13166 -0.26128" rpy="0 0 0"/>
     <geometry>
       <mesh filename="package://robotic_arm_description/meshes/gripper_base_v8_1.stl" scale="0.001 0.001 0.001"/>
@@ -209,10 +210,10 @@
 <link name="gripper_gear_1_v2_1">
   <inertial>
-    <origin xyz="-0.0005644997090397674 -0.005402189148709768 0.0020000001341104467" rpy="0 0 0"/>
+    <origin xyz="-0.0005644997090396842 -0.005402189148709879 0.002000000134110169" rpy="0 0 0"/>
     <mass value="0.0029250313733063305"/>
-    <inertia ixx="0.0" iyy="0.0" izz="1e-06" ixy="0.0" iyz="-0.0" ixz="0.0"/>
-  </inertial>
-  <visual>
-    <origin xyz="-0.3274 0.23966 -0.27528" rpy="0 0 0"/>
+    <inertia ixx="0.0" iyy="0.0" izz="1e-06" ixy="0.0" iyz="0.0" ixz="0.0"/>
+  </inertial>
+  <visual>
+    <origin xyz="-0.0299 0.16966 -0.27528" rpy="0 0 0"/>
     <geometry>
       <mesh filename="package://robotic_arm_description/meshes/gripper_gear_1_v2_1.stl" scale="0.001 0.001 0.001"/>
@@ -221,5 +222,5 @@
   </visual>
   <collision>
-    <origin xyz="-0.3274 0.23966 -0.27528" rpy="0 0 0"/>
+    <origin xyz="-0.0299 0.16966 -0.27528" rpy="0 0 0"/>
     <geometry>
       <mesh filename="package://robotic_arm_description/meshes/gripper_gear_1_v2_1.stl" scale="0.001 0.001 0.001"/>
@@ -229,90 +230,90 @@
 <link name="gripper_v3_1">
   <inertial>
-    <origin xyz="0.004099853901063655 -0.02653931048241409 0.004250000134110421" rpy="0 0 0"/>
+    <origin xyz="0.004099853901063728 -0.026539310482414202 0.0042500001341101434" rpy="0 0 0"/>
+    <mass value="0.005742804742280986"/>
+    <inertia ixx="2e-06" iyy="0.0" izz="2e-06" ixy="0.0" iyz="0.0" ixz="-0.0"/>
+  </inertial>
+  <visual>
+    <origin xyz="-0.0299 0.20041 -0.27928" rpy="0 0 0"/>
+    <geometry>
+      <mesh filename="package://robotic_arm_description/meshes/gripper_v3_1.stl" scale="0.001 0.001 0.001"/>
+    </geometry>
+    <material name="pa_12_nylon_pa_603cf_with_eos_p_3d_printers"/>
+  </visual>
+  <collision>
+    <origin xyz="-0.0299 0.20041 -0.27928" rpy="0 0 0"/>
+    <geometry>
+      <mesh filename="package://robotic_arm_description/meshes/gripper_v3_1.stl" scale="0.001 0.001 0.001"/>
+    </geometry>
+  </collision>
+</link>
+<link name="gripper_v3_2">
+  <inertial>
+    <origin xyz="0.004099853901063589 -0.026539310482414286 -0.004249999865889864" rpy="0 0 0"/>
     <mass value="0.005742804742280986"/>
     <inertia ixx="2e-06" iyy="0.0" izz="2e-06" ixy="0.0" iyz="0.0" ixz="0.0"/>
   </inertial>
   <visual>
-    <origin xyz="-0.3274 0.27041 -0.27928" rpy="0 0 0"/>
-    <geometry>
-      <mesh filename="package://robotic_arm_description/meshes/gripper_v3_1.stl" scale="0.001 0.001 0.001"/>
-    </geometry>
-    <material name="pa_12_nylon_pa_603cf_with_eos_p_3d_printers"/>
-  </visual>
-  <collision>
-    <origin xyz="-0.3274 0.27041 -0.27928" rpy="0 0 0"/>
-    <geometry>
-      <mesh filename="package://robotic_arm_description/meshes/gripper_v3_1.stl" scale="0.001 0.001 0.001"/>
-    </geometry>
-  </collision>
-</link>
-<link name="gripper_v3_2">
-  <inertial>
-    <origin xyz="0.004099853901063488 -0.026539310482414202 -0.004249999865889642" rpy="0 0 0"/>
+    <origin xyz="-0.0299 0.20041 -0.27528" rpy="0 0 0"/>
+    <geometry>
+      <mesh filename="package://robotic_arm_description/meshes/gripper_v3_2.stl" scale="0.001 0.001 0.001"/>
+    </geometry>
+    <material name="pa_12_nylon_pa_603cf_with_eos_p_3d_printers"/>
+  </visual>
+  <collision>
+    <origin xyz="-0.0299 0.20041 -0.27528" rpy="0 0 0"/>
+    <geometry>
+      <mesh filename="package://robotic_arm_description/meshes/gripper_v3_2.stl" scale="0.001 0.001 0.001"/>
+    </geometry>
+  </collision>
+</link>
+<link name="gripper_gear_2_v2_1">
+  <inertial>
+    <origin xyz="0.0005811920264956459 -0.005561932438407968 0.0020000001341103357" rpy="0 0 0"/>
+    <mass value="0.0028410220441566826"/>
+    <inertia ixx="0.0" iyy="0.0" izz="0.0" ixy="-0.0" iyz="0.0" ixz="0.0"/>
+  </inertial>
+  <visual>
+    <origin xyz="-0.003 0.16966 -0.27528" rpy="0 0 0"/>
+    <geometry>
+      <mesh filename="package://robotic_arm_description/meshes/gripper_gear_2_v2_1.stl" scale="0.001 0.001 0.001"/>
+    </geometry>
+    <material name="opaque160160160"/>
+  </visual>
+  <collision>
+    <origin xyz="-0.003 0.16966 -0.27528" rpy="0 0 0"/>
+    <geometry>
+      <mesh filename="package://robotic_arm_description/meshes/gripper_gear_2_v2_1.stl" scale="0.001 0.001 0.001"/>
+    </geometry>
+  </collision>
+</link>
+<link name="gripper_v3_3">
+  <inertial>
+    <origin xyz="-0.004099853901064021 -0.026539310482414313 -0.004249999865889698" rpy="0 0 0"/>
     <mass value="0.005742804742280986"/>
-    <inertia ixx="2e-06" iyy="0.0" izz="2e-06" ixy="0.0" iyz="-0.0" ixz="0.0"/>
-  </inertial>
-  <visual>
-    <origin xyz="-0.3274 0.27041 -0.27528" rpy="0 0 0"/>
-    <geometry>
-      <mesh filename="package://robotic_arm_description/meshes/gripper_v3_2.stl" scale="0.001 0.001 0.001"/>
-    </geometry>
-    <material name="pa_12_nylon_pa_603cf_with_eos_p_3d_printers"/>
-  </visual>
-  <collision>
-    <origin xyz="-0.3274 0.27041 -0.27528" rpy="0 0 0"/>
-    <geometry>
-      <mesh filename="package://robotic_arm_description/meshes/gripper_v3_2.stl" scale="0.001 0.001 0.001"/>
-    </geometry>
-  </collision>
-</link>
-<link name="gripper_gear_2_v2_1">
-  <inertial>
-    <origin xyz="0.0005811920264957027 -0.005561932438407885 0.0020000001341104467" rpy="0 0 0"/>
-    <mass value="0.0028410220441566826"/>
-    <inertia ixx="0.0" iyy="0.0" izz="0.0" ixy="-0.0" iyz="-0.0" ixz="-0.0"/>
-  </inertial>
-  <visual>
-    <origin xyz="-0.3005 0.23966 -0.27528" rpy="0 0 0"/>
-    <geometry>
-      <mesh filename="package://robotic_arm_description/meshes/gripper_gear_2_v2_1.stl" scale="0.001 0.001 0.001"/>
-    </geometry>
-    <material name="opaque160160160"/>
-  </visual>
-  <collision>
-    <origin xyz="-0.3005 0.23966 -0.27528" rpy="0 0 0"/>
-    <geometry>
-      <mesh filename="package://robotic_arm_description/meshes/gripper_gear_2_v2_1.stl" scale="0.001 0.001 0.001"/>
-    </geometry>
-  </collision>
-</link>
-<link name="gripper_v3_3">
-  <inertial>
-    <origin xyz="-0.004099853901063988 -0.026539310482414258 -0.0042499998658895866" rpy="0 0 0"/>
+    <inertia ixx="2e-06" iyy="0.0" izz="2e-06" ixy="-0.0" iyz="0.0" ixz="-0.0"/>
+  </inertial>
+  <visual>
+    <origin xyz="-0.003 0.20041 -0.27528" rpy="0 0 0"/>
+    <geometry>
+      <mesh filename="package://robotic_arm_description/meshes/gripper_v3_3.stl" scale="0.001 0.001 0.001"/>
+    </geometry>
+    <material name="pa_12_nylon_pa_603cf_with_eos_p_3d_printers"/>
+  </visual>
+  <collision>
+    <origin xyz="-0.003 0.20041 -0.27528" rpy="0 0 0"/>
+    <geometry>
+      <mesh filename="package://robotic_arm_description/meshes/gripper_v3_3.stl" scale="0.001 0.001 0.001"/>
+    </geometry>
+  </collision>
+</link>
+<link name="gripper_v3_4">
+  <inertial>
+    <origin xyz="-0.004099853901064242 -0.026539310482414286 0.004250000134110088" rpy="0 0 0"/>
     <mass value="0.005742804742280986"/>
     <inertia ixx="2e-06" iyy="0.0" izz="2e-06" ixy="-0.0" iyz="-0.0" ixz="-0.0"/>
   </inertial>
   <visual>
-    <origin xyz="-0.3005 0.27041 -0.27528" rpy="0 0 0"/>
-    <geometry>
-      <mesh filename="package://robotic_arm_description/meshes/gripper_v3_3.stl" scale="0.001 0.001 0.001"/>
-    </geometry>
-    <material name="pa_12_nylon_pa_603cf_with_eos_p_3d_printers"/>
-  </visual>
-  <collision>
-    <origin xyz="-0.3005 0.27041 -0.27528" rpy="0 0 0"/>
-    <geometry>
-      <mesh filename="package://robotic_arm_description/meshes/gripper_v3_3.stl" scale="0.001 0.001 0.001"/>
-    </geometry>
-  </collision>
-</link>
-<link name="gripper_v3_4">
-  <inertial>
-    <origin xyz="-0.00409985390106421 -0.026539310482414202 0.004250000134110199" rpy="0 0 0"/>
-    <mass value="0.005742804742280986"/>
-    <inertia ixx="2e-06" iyy="0.0" izz="2e-06" ixy="-0.0" iyz="0.0" ixz="-0.0"/>
-  </inertial>
-  <visual>
-    <origin xyz="-0.3005 0.27041 -0.27928" rpy="0 0 0"/>
+    <origin xyz="-0.003 0.20041 -0.27928" rpy="0 0 0"/>
     <geometry>
       <mesh filename="package://robotic_arm_description/meshes/gripper_v3_4.stl" scale="0.001 0.001 0.001"/>
@@ -321,5 +322,5 @@
   </visual>
   <collision>
-    <origin xyz="-0.3005 0.27041 -0.27928" rpy="0 0 0"/>
+    <origin xyz="-0.003 0.20041 -0.27928" rpy="0 0 0"/>
     <geometry>
       <mesh filename="package://robotic_arm_description/meshes/gripper_v3_4.stl" scale="0.001 0.001 0.001"/>
@@ -328,5 +329,5 @@
 </link>
 <joint name="rigid_1" type="fixed">
-  <origin xyz="0.2975 0.0 0.015" rpy="0 0 0"/>
+  <origin xyz="0.0 0.07 0.015" rpy="0 0 0"/>
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
File: src/robotic_arm_description/urdf/robotic_arm_controllers.xacro (robot description, xacro)
@@ -2,6 +2,6 @@
 <robot xmlns:xacro="http://www.ros.org/wiki/xacro" name="robotic_arm">
 <xacro:property name="gripper_angle" value="0.7854"/>
- <xacro:property name="PI" value="3.14159"/>
- <ros2_control type = "system" name = "RoboticArmSystem">
+<xacro:property name="PI" value="3.14159"/>
+<ros2_control type = "system" name = "RoboticArmSystem">
     <hardware>
         <plugin>gazebo_ros2_control/GazeboSystem</plugin>
