Commit message: Added The msgs package

File: src/robotic_arm_description/urdf/robotic_arm.xacro (robot description, xacro)
@@ -4,8 +4,9 @@
 <xacro:include filename="$(find robotic_arm_description)/urdf/robotic_arm.trans" />
 <xacro:include filename="$(find robotic_arm_description)/urdf/robotic_arm_gazebo.xacro"/>
-<xacro:include filename="$(find robotic_arm_description)/urdf/robotic_arm.gazebo.xacro"/>
 <xacro:include filename="$(find robotic_arm_description)/urdf/robotic_arm_controllers.xacro"/>
 <!-- Properties -->
 <xacro:property name="PI" value="1.570796"/>
+<!-- Links -->
+<link name = "world"/>
 <link name="base_link">
   <inertial>
@@ -328,4 +329,10 @@
   </collision>
 </link>
+<!-- Joints -->
+<joint name = "virtual_joint" type= "fixed">
+  <origin xyz="0.0 0.0 0.0" rpy="0.0 0.0 0.0"/>
+  <parent link="world"/>
+  <child link="base_link"/>
+</joint>
 <joint name="rigid_1" type="fixed">
   <origin xyz="0.0 0.07 0.015" rpy="0 0 0"/>
@@ -337,11 +344,7 @@
   <parent link="base_v2_1"/>
   <child link="waist_v6_1"/>
-  <axis xyz="0.0 -0.0 1.0"/>
+  <axis xyz="0.0 0.0 1.0"/>
+  <dynamics damping="10.0" friction="5.0"/>
   <limit upper="1.570796" lower="-1.570796" effort="100" velocity="100"/>
-</joint>
-<joint name="rigid_2" type="fixed">
-  <origin xyz="-0.018 -0.027168 0.046467" rpy="0 0 0"/>
-  <parent link="waist_v6_1"/>
-  <child link="servomotormg996r_v2_2"/>
 </joint>
 <joint name="waist_link1_joint" type="revolute">
@@ -350,4 +353,5 @@
   <child link="link_1_v5_1"/>
   <axis xyz="1.0 0.0 0.0"/>
+  <dynamics damping="10.0" friction="5.0"/>
   <limit upper="1.570796" lower="-1.570796" effort="100" velocity="100"/>
 </joint>
@@ -356,21 +360,7 @@
   <parent link="link_1_v5_1"/>
   <child link="link_2a_v4_1"/>
-  <axis xyz="-1.0 0.0 -0.0"/>
+  <axis xyz="-1.0 0.0 0.0"/>
+  <dynamics damping="10.0" friction="5.0"/>
   <limit upper="3.141593" lower="0.0" effort="100" velocity="100"/>
-</joint>
-<joint name="rigid_3" type="fixed">
-  <origin xyz="0.008 -0.08975 0.0" rpy="0 0 0"/>
-  <parent link="link_2a_v4_1"/>
-  <child link="link_2b_v4_1"/>
-</joint>
-<joint name="rigid_4" type="fixed">
-  <origin xyz="-0.011 -0.03475 -0.005" rpy="0 0 0"/>
-  <parent link="link_2a_v4_1"/>
-  <child link="servomotormg996r_v2_3"/>
-</joint>
-<joint name="rigid_5" type="fixed">
-  <origin xyz="-0.0105 -0.0368 0.0" rpy="0 0 0"/>
-  <parent link="link_2b_v4_1"/>
-  <child link="servomotormicro9g_v2_1"/>
 </joint>
 <joint name="link2_gripperbase_joint" type="revolute">
@@ -379,5 +369,26 @@
   <child link="gripper_base_v8_1"/>
   <axis xyz="1.0 -0.0 0.0"/>
+  <dynamics damping="10.0" friction="5.0"/>
   <limit upper="1.570796" lower="-1.570796" effort="100" velocity="100"/>
+</joint>
+<joint name="rigid_2" type="fixed">
+  <origin xyz="-0.018 -0.027168 0.046467" rpy="0 0 0"/>
+  <parent link="waist_v6_1"/>
+  <child link="servomotormg996r_v2_2"/>
+</joint>
+<joint name="rigid_3" type="fixed">
+  <origin xyz="0.008 -0.08975 0.0" rpy="0 0 0"/>
+  <parent link="link_2a_v4_1"/>
+  <child link="link_2b_v4_1"/>
+</joint>
+<joint name="rigid_4" type="fixed">
+  <origin xyz="-0.011 -0.03475 -0.005" rpy="0 0 0"/>
+  <parent link="link_2a_v4_1"/>
+  <child link="servomotormg996r_v2_3"/>
+</joint>
+<joint name="rigid_5" type="fixed">
+  <origin xyz="-0.0105 -0.0368 0.0" rpy="0 0 0"/>
+  <parent link="link_2b_v4_1"/>
+  <child link="servomotormicro9g_v2_1"/>
 </joint>
 <joint name="rigid_6" type="fixed">
@@ -396,4 +407,5 @@
   <child link="gripper_gear_2_v2_1"/>
   <axis xyz="0.0 0.0 -1.0"/>
+  <dynamics damping="10.0" friction="5.0"/>
   <limit upper="${gripper_angle}" lower="0.0" effort="100" velocity="100"/>
 </joint>
@@ -403,4 +415,5 @@
   <child link="gripper_gear_1_v2_1"/>
   <axis xyz="-0.0 -0.0 1.0"/>
+  <dynamics damping="10.0" friction="5.0"/>
   <mimic joint = "right_gripper_joint" multiplier = "1.0"/>
   <limit upper = "-${gripper_angle}" lower="0.0" effort="100" velocity="100"/>

File: src/robotic_arm_description/urdf/robotic_arm_controllers.xacro (robot description, xacro)
@@ -24,5 +24,5 @@
     <joint name="link1_link2_joint">
         <command_interface name="position">
-            <param name = "min">0,0</param>
+            <param name = "min">0.0</param>
             <param name = "max">${PI}</param>
         </command_interface>

File: src/robotic_arm_description/urdf/robotic_arm_gazebo.xacro (robot description, xacro)
@@ -1,5 +1,13 @@
 <?xml version="1.0" encoding = "UTF-8"?>
-<robot xmlns:xacro="http://www.ros.org/wiki/xacro" name="robotic_arm">
-    <gazebo>
+<robot name="robotic_arm" xmlns:xacro="http://www.ros.org/wiki/xacro" >
+<xacro:property name="base_color" value = "Gazebo/Oak"/>
+<xacro:property name="waist_color" value = "Gazebo/FlatBlack" />
+<xacro:property name="link_1_color" value = "Gazebo/FlatBlack"/>
+<xacro:property name="link_2_color" value = "Gazebo/FlatBlack" />
+<xacro:property name="gripper_base_color" value = "Gazebo/FlatBlack" />
+<xacro:property name="motor_color" value="Gazebo/Blue" />
+<xacro:property name="gripper_gears" value="GazeboGrey"/>
+<xacro:property name="gripper_color" value="Gazebo/DarkGrey" />
+<gazebo>
         <plugin filename="libgazebo_ros2_control.so" name="gazebo_ros2_control">
             <robot_param> robot_description</robot_param>
@@ -7,4 +15,107 @@
             <parameters>$(find robotic_arm_controllers)/config/robot_arm_controllers.yaml</parameters>
         </plugin>
-    </gazebo>
+</gazebo>
+<gazebo reference="base_link">
+  <material>${base_color}</material>
+  <mu1>0.2</mu1>
+  <mu2>0.2</mu2>
+  <self_collide>true</self_collide>
+  <gravity>true</gravity>
+</gazebo>
+<gazebo reference="base_v2_1">
+  <material>${waist_color}</material>
+  <mu1>0.2</mu1>
+  <mu2>0.2</mu2>
+  <self_collide>true</self_collide>
+</gazebo>
+<gazebo reference="waist_v6_1">
+  <material>${waist_color}</material>
+  <mu1>0.2</mu1>
+  <mu2>0.2</mu2>
+  <self_collide>true</self_collide>
+</gazebo>
+<gazebo reference="link_1_v5_1">
+  <material>${link_1_color}</material>
+  <mu1>0.2</mu1>
+  <mu2>0.2</mu2>
+  <self_collide>true</self_collide>
+</gazebo>
+<gazebo reference="link_2a_v4_1">
+  <material>${link_2_color}</material>
+  <mu1>0.2</mu1>
+  <mu2>0.2</mu2>
+  <self_collide>true</self_collide>
+</gazebo>
+<gazebo reference="link_2b_v4_1">
+  <material>${link_2_color}</material>
+  <mu1>0.2</mu1>
+  <mu2>0.2</mu2>
+  <self_collide>true</self_collide>
+</gazebo>
+<gazebo reference="gripper_base_v8_1">
+  <material>${gripper_base_color}</material>
+  <mu1>0.2</mu1>
+  <mu2>0.2</mu2>
+  <self_collide>true</self_collide>
+</gazebo>
+<gazebo reference="servomotormicro9g_v2_1">
+  <material>${motor_color}</material>
+  <mu1>0.2</mu1>
+  <mu2>0.2</mu2>
+  <self_collide>true</self_collide>
+</gazebo>
+<gazebo reference="servomotormg996r_v2_2">
+  <material>${motor_color}</material>
+  <mu1>0.2</mu1>
+  <mu2>0.2</mu2>
+  <self_collide>true</self_collide>
+</gazebo>
+<gazebo reference="servomotormicro9g_v2_2">
+  <material>${motor_color}</material>
+  <mu1>0.2</mu1>
+  <mu2>0.2</mu2>
+  <self_collide>true</self_collide>
+</gazebo>
+<gazebo reference="servomotormg996r_v2_3">
+  <material>${motor_color}</material>
+  <mu1>0.2</mu1>
+  <mu2>0.2</mu2>
+  <self_collide>true</self_collide>
+</gazebo>
+<gazebo reference="gripper_gear_1_v2_1">
+  <material>${gripper_gears}</material>
+  <mu1>0.2</mu1>
+  <mu2>0.2</mu2>
+  <self_collide>true</self_collide>
+</gazebo>
+<gazebo reference="gripper_gear_2_v2_1">
+  <material>${gripper_gears}</material>
+  <mu1>0.2</mu1>
+  <mu2>0.2</mu2>
+  <self_collide>true</self_collide>
+</gazebo>
+<gazebo reference="gripper_v3_1">
+  <material>${gripper_color}</material>
+  <mu1>0.2</mu1>
+  <mu2>0.2</mu2>
+  <self_collide>true</self_collide>
+</gazebo>
+<gazebo reference="gripper_v3_2">
+  <material>${gripper_color}</material>
+  <mu1>0.2</mu1>
+  <mu2>0.2</mu2>
+  <self_collide>true</self_collide>
+</gazebo>
+<gazebo reference="gripper_v3_3">
+  <material>${gripper_color}</material>
+  <mu1>0.2</mu1>
+  <mu2>0.2</mu2>
+  <self_collide>true</self_collide>
+</gazebo>
+<gazebo reference="gripper_v3_4">
+  <material>${gripper_color}</material>
+  <mu1>0.2</mu1>
+  <mu2>0.2</mu2>
+  <self_collide>true</self_collide>
+</gazebo>
 </robot>

Commit message: added roboticstoolbox python file

File: src/robotic_arm_description/urdf/robotic_arm.xacro (robot description, xacro)
@@ -184,4 +184,5 @@
   <child link="waist"/>
   <axis xyz="0.0 0.0 1.0"/>
+  <dynamics damping="10.0" friction="2.0"/>
   <limit upper="1.570796" lower="-1.570796" effort="100" velocity="100"/>
 </joint>
@@ -191,4 +192,5 @@
   <child link="link_1"/>
   <axis xyz="1.0 0.0 -0.0"/>
+  <dynamics damping="10.0" friction="2.0"/>
   <limit upper="1.570796" lower="-1.570796" effort="100" velocity="100"/>
 </joint>
@@ -198,4 +200,5 @@
   <child link="link_2"/>
   <axis xyz="-1.0 0.0 -0.0"/>
+  <dynamics damping="10.0" friction="2.0"/>
   <limit upper="3.141593" lower="0.0" effort="100" velocity="100"/>
 </joint>
@@ -205,4 +208,5 @@
   <child link="gripper_base"/>
   <axis xyz="1.0 0.0 0.0"/>
+  <dynamics damping="10.0" friction="2.0"/>
   <limit upper="1.570796" lower="-1.570796" effort="100" velocity="100"/>
 </joint>
@@ -212,4 +216,5 @@
   <child link="gripper_finger_2"/>
   <axis xyz="0.0 0.0 -1.0"/>
+  <dynamics damping="10.0" friction="2.0"/>
   <limit upper="0.785398" lower="0.0" effort="100" velocity="100"/>
 </joint>
@@ -219,4 +224,5 @@
   <child link="gripper_finger_1"/>
   <axis xyz="-0.0 -0.0 1.0"/>
+  <dynamics damping="10.0" friction="2.0"/>
   <mimic joint = "right_gripper_joint" multiplier = "1.0"/>
   <limit upper="-0.785398" lower="0.0" effort="100" velocity="100"/>

File: src/robotic_arm_description/urdf/robotic_arm_urdf.urdf (robot description, URDF)
Before this commit: robot robotic_arm, 9 links, 8 joints
Joints:
- joint left_gripper_joint: axis -0.0 -0.0 1.0 -> 0.0 0.0 1.0
- joint link1_link2_joint: axis -1.0 0.0 -0.0 -> -1.0 0.0 0.0
- joint waist_link1_joint: axis 1.0 0.0 -0.0 -> 1.0 0.0 0.0
